Commit message: SMall fixes to improve simualtion behaviour

File: src/leo_gazebo/description/leo_sim.xacro (robot description, xacro)
@@ -53,5 +53,5 @@
         <child link="wheel_fl" />
         <axis xyz="0 0 1" />
-        <dynamics damping="0.7" friction="1.0" />
+        <dynamics damping="0.5" friction="0.80" />
     </joint>
     <link name="wheel_fr">
@@ -77,5 +77,5 @@
         <child link="wheel_fr" />
         <axis xyz="0 0 1" />
-        <dynamics damping="0.7" friction="1.0" />
+        <dynamics damping="0.5" friction="0.80" />
     </joint>
     <link name="wheel_rl">
@@ -101,5 +101,5 @@
         <child link="wheel_rl" />
         <axis xyz="0 0 1" />
-        <dynamics damping="0.7" friction="1.0" />
+        <dynamics damping="0.5" friction="0.80" />
     </joint>
     <link name="wheel_rr">
@@ -125,5 +125,5 @@
         <child link="wheel_rr" />
         <axis xyz="0 0 1" />
-        <dynamics damping="0.7" friction="1.0" />
+        <dynamics damping="0.5" friction="0.80" />
     </joint>
     <!-- Jetson Mount -->
