Commit message: Small changes synced automatically

File: src/leo_description/description/leo_sim.xacro (robot description, xacro)
@@ -27,5 +27,5 @@
         <inertial>
             <mass value="10" />
-            <inertia ixx="0.01" ixy="0" ixz="0" iyy="0.01" iyz="0" izz="0.01" />
+            <inertia ixx="0.1" ixy="0" ixz="0" iyy="0.1" iyz="0" izz="0.15" />
         </inertial>
     </link>
@@ -53,5 +53,5 @@
         <child link="wheel_fl" />
         <axis xyz="0 0 1" />
-        <dynamics damping="0.5" friction="0.80" />
+        <dynamics damping="0.0" friction="0.0" />
     </joint>
     <link name="wheel_fr">
@@ -77,5 +77,5 @@
         <child link="wheel_fr" />
         <axis xyz="0 0 1" />
-        <dynamics damping="0.5" friction="0.80" />
+        <dynamics damping="0.0" friction="0.0" />
     </joint>
     <link name="wheel_rl">
@@ -101,5 +101,5 @@
         <child link="wheel_rl" />
         <axis xyz="0 0 1" />
-        <dynamics damping="0.5" friction="0.80" />
+        <dynamics damping="0.0" friction="0.0" />
     </joint>
     <link name="wheel_rr">
@@ -125,5 +125,5 @@
         <child link="wheel_rr" />
         <axis xyz="0 0 1" />
-        <dynamics damping="0.5" friction="0.80" />
+        <dynamics damping="0.0" friction="0.0" />
     </joint>
     <!-- Jetson Mount -->
@@ -185,6 +185,6 @@
             <wheel_separation>0.354</wheel_separation>
             <wheel_diameter>0.129</wheel_diameter>
-            <max_wheel_torque>200</max_wheel_torque>
-            <max_wheel_acceleration>10.0</max_wheel_acceleration>
+            <max_wheel_torque>1000</max_wheel_torque>
+            <max_wheel_acceleration>100.0</max_wheel_acceleration>
             <command_topic>cmd_vel</command_topic>
             <odometry_topic>odom</odometry_topic>
@@ -201,29 +201,29 @@
     <gazebo reference="wheel_fl">
         <material>Gazebo/Black</material>
-        <mu1>1.5</mu1>
-        <mu2>1.5</mu2>
-        <kp>1000000.0</kp>
-        <kd>1.0</kd>
+        <mu1>10.0</mu1>
+        <mu2>10.0</mu2>
+        <kp>1000000.0</kp>
+        <kd>10.0</kd>
     </gazebo>
     <gazebo reference="wheel_fr">
         <material>Gazebo/Black</material>
-        <mu1>1.5</mu1>
-        <mu2>1.5</mu2>
-        <kp>1000000.0</kp>
-        <kd>1.0</kd>
+        <mu1>10.0</mu1>
+        <mu2>10.0</mu2>
+        <kp>1000000.0</kp>
+        <kd>10.0</kd>
     </gazebo>
     <gazebo reference="wheel_rl">
         <material>Gazebo/Black</material>
-        <mu1>1.5</mu1>
-        <mu2>1.5</mu2>
-        <kp>1000000.0</kp>
-        <kd>1.0</kd>
+        <mu1>10.0</mu1>
+        <mu2>10.0</mu2>
+        <kp>1000000.0</kp>
+        <kd>10.0</kd>
     </gazebo>
     <gazebo reference="wheel_rr">
         <material>Gazebo/Black</material>
-        <mu1>1.5</mu1>
-        <mu2>1.5</mu2>
-        <kp>1000000.0</kp>
-        <kd>1.0</kd>
+        <mu1>10.0</mu1>
+        <mu2>10.0</mu2>
+        <kp>1000000.0</kp>
+        <kd>10.0</kd>
     </gazebo>
     <gazebo reference="velodyne">

File: src/leo_description/description/wheels.xacro (robot description, xacro)
@@ -7,96 +7,96 @@
             <visual>
                 <geometry>
-                    <cylinder radius="0.0645" length="0.065"/>
+                    <cylinder radius="0.0645" length="0.065" />
                 </geometry>
-                <material name="black"/>
+                <material name="black" />
             </visual>
             <collision>
                 <geometry>
-                    <cylinder radius="0.0645" length="0.065"/>
+                    <cylinder radius="0.0645" length="0.065" />
                 </geometry>
             </collision>
             <inertial>
-                <mass value="0.5"/>
-                <inertia ixx="0.01" ixy="0" ixz="0" iyy="0.01" iyz="0" izz="0.01"/>
+                <mass value="0.5" />
+                <inertia ixx="0.01" ixy="0" ixz="0" iyy="0.01" iyz="0" izz="0.01" />
             </inertial>
         </link>
         <joint name="wheel_fl_chassis" type="continuous">
-            <origin xyz="0.1475 0.177 0.0" rpy="-1.5708 0 0"/>
-            <parent link="${parent}"/>
-            <child link="wheel_fl"/>
-            <axis xyz="0 0 1"/>
-            <dynamics damping="0.7" friction="1.0"/>
+            <origin xyz="0.1475 0.177 0.0" rpy="-1.5708 0 0" />
+            <parent link="${parent}" />
+            <child link="wheel_fl" />
+            <axis xyz="0 0 1" />
+            <dynamics damping="0.7" friction="1.0" />
         </joint>
         <link name="wheel_fr">
             <visual>
                 <geometry>
-                    <cylinder radius="0.0645" length="0.065"/>
+                    <cylinder radius="0.0645" length="0.065" />
                 </geometry>
-                <material name="black"/>
+                <material name="black" />
             </visual>
             <collision>
                 <geometry>
-                    <cylinder radius="0.0645" length="0.065"/>
+                    <cylinder radius="0.0645" length="0.065" />
                 </geometry>
             </collision>
             <inertial>
-                <mass value="0.5"/>
-                <inertia ixx="0.01" ixy="0" ixz="0" iyy="0.01" iyz="0" izz="0.01"/>
+                <mass value="0.5" />
+                <inertia ixx="0.01" ixy="0" ixz="0" iyy="0.01" iyz="0" izz="0.01" />
             </inertial>
         </link>
         <joint name="wheel_fr_chassis" type="continuous">
-            <origin xyz="0.1475 -0.177 0.0" rpy="-1.5708 0 0"/>
-            <parent link="${parent}"/>
-            <child link="wheel_fr"/>
-            <axis xyz="0 0 1"/>
-            <dynamics damping="0.7" friction="1.0"/>
+            <origin xyz="0.1475 -0.177 0.0" rpy="-1.5708 0 0" />
+            <parent link="${parent}" />
+            <child link="wheel_fr" />
+            <axis xyz="0 0 1" />
+            <dynamics damping="0.7" friction="1.0" />
         </joint>
         <link name="wheel_rl">
             <visual>
                 <geometry>
-                    <cylinder radius="0.0645" length="0.065"/>
+                    <cylinder radius="0.0645" length="0.065" />
                 </geometry>
-                <material name="black"/>
+                <material name="black" />
             </visual>
             <collision>
                 <geometry>
-                    <cylinder radius="0.0645" length="0.065"/>
+                    <cylinder radius="0.0645" length="0.065" />
                 </geometry>
             </collision>
             <inertial>
-                <mass value="0.5"/>
-                <inertia ixx="0.01" ixy="0" ixz="0" iyy="0.01" iyz="0" izz="0.01"/>
+                <mass value="0.5" />
+                <inertia ixx="0.01" ixy="0" ixz="0" iyy="0.01" iyz="0" izz="0.01" />
             </inertial>
         </link>
         <joint name="wheel_rl_chassis" type="continuous">
-            <origin xyz="-0.1475 0.177 0.0" rpy="-1.5708 0 0"/>
-            <parent link="${parent}"/>
-            <child link="wheel_rl"/>
-            <axis xyz="0 0 1"/>
-            <dynamics damping="0.7" friction="1.0"/>
+            <origin xyz="-0.1475 0.177 0.0" rpy="-1.5708 0 0" />
+            <parent link="${parent}" />
+            <child link="wheel_rl" />
+            <axis xyz="0 0 1" />
+            <dynamics damping="0.7" friction="1.0" />
         </joint>
         <link name="wheel_rr">
             <visual>
                 <geometry>
-                    <cylinder radius="0.0645" length="0.065"/>
+                    <cylinder radius="0.0645" length="0.065" />
                 </geometry>
-                <material name="black"/>
+                <material name="black" />
             </visual>
             <collision>
                 <geometry>
-                    <cylinder radius="0.0645" length="0.065"/>
+                    <cylinder radius="0.0645" length="0.065" />
                 </geometry>
             </collision>
             <inertial>
-                <mass value="0.5"/>
-                <inertia ixx="0.01" ixy="0" ixz="0" iyy="0.01" iyz="0" izz="0.01"/>
+                <mass value="0.5" />
+                <inertia ixx="0.01" ixy="0" ixz="0" iyy="0.01" iyz="0" izz="0.01" />
             </inertial>
         </link>
         <joint name="wheel_rr_chassis" type="continuous">
-            <origin xyz="-0.1475 -0.177 0.0" rpy="-1.5708 0 0"/>
-            <parent link="${parent}"/>
-            <child link="wheel_rr"/>
-            <axis xyz="0 0 1"/>
-            <dynamics damping="0.7" friction="1.0"/>
+            <origin xyz="-0.1475 -0.177 0.0" rpy="-1.5708 0 0" />
+            <parent link="${parent}" />
+            <child link="wheel_rr" />
+            <axis xyz="0 0 1" />
+            <dynamics damping="0.7" friction="1.0" />
         </joint>
     </xacro:macro>
